Commit message: MZ12H urdf updated

File: urdf/MZ12H.urdf (robot description, URDF)
Before this commit: robot MZ12H, 10 links, 9 joints
Links:
- link link2: mass 7.26567587988546 -> 7.26567581405818
- link link3: mass 13.4942571777588 -> 13.494257553147
- link link4: mass 7.6088166218264 -> 7.60881664037561
- link link4_left_logo: mass 0.000628941851328343 -> 0.000628941851328278
- link link4_right_logo: mass 7.6094427354956 -> 7.60944275405364
- link link5: mass 0.560948385919128 -> 0.560948386973578
- link link6: mass 0.0439410372876388 -> 0.0439410372876389
Joints:
- joint j1_logo_left: axis 0 0 1 -> 0 0 0; origin xyz=0 0.01 0 rpy=0 0 0 -> xyz=0 0 0.008 rpy=0 0 0
- joint j2: limit (none) -> lower=0 upper=0 effort=0 velocity=0; type continuous -> revolute
- joint j4_left_logo: origin xyz=0.44454 0.01 0 rpy=0 0 0 -> xyz=0.444539076030978 0 0 rpy=0 0 0
- joint j4_logo_right: origin xyz=0.44454 0 0 rpy=0 0 0 -> xyz=0.444539076030978 0 0 rpy=0 0 0
- joint j5: origin xyz=0.44454 0.01 0 rpy=0 0 0 -> xyz=0.44454 0 0 rpy=0 0 0
- joint j6: origin xyz=0.082 -0.01 0 rpy=0 0 0 -> xyz=0.082 0 0 rpy=0 0 0

Commit message: jt5

File: urdf/MZ12H.urdf (robot description, URDF)
Before this commit: robot MZ12H, 10 links, 9 joints
Joints:
- joint j5: limit lower=0 upper=0 effort=0 velocity=0 -> lower=-3.14 upper=3.14 effort=10 velocity=1

Commit message: axis xyz fix

File: urdf/MZ12H.urdf (robot description, URDF)
Before this commit: robot MZ12H, 10 links, 9 joints
Joints:
- joint j2: axis 1 -1 0 -> 0 -1 0

Commit message: faah

File: urdf/MZ12H.urdf (robot description, URDF)
Before this commit: robot MZ12H, 10 links, 9 joints
Links:
- removed link link1_logo_left
- removed link link4_left_logo
- removed link link4_right_logo
- added link link1_logo, mass 0.000262575877525974; collision mesh filename=package://MZ12H/meshes/link1_logo.STL; visual mesh filename=package://MZ12H/meshes/link1_logo.STL
- added link link4_logo_left, mass 0.000628941851328052; collision mesh filename=package://MZ12H/meshes/link4_logo_left.STL; visual mesh filename=package://MZ12H/meshes/link4_logo_left.STL
- added link link4_logo_right, mass 7.60944232108211; collision mesh filename=package://MZ12H/meshes/link4_logo_right.STL; visual mesh filename=package://MZ12H/meshes/link4_logo_right.STL
- link link1: mass 20.9171454922225 -> 20.917144981739
- link link2: mass 7.26567581405818 -> 7.26567570560942
- link link3: mass 13.494257553147 -> 13.4942572400188
- link link4: mass 7.60881664037561 -> 7.60881636541159
- link link5: mass 0.560948386973578 -> 0.560948383901603
- link link6: mass 0.0439410372876389 -> 0.0439410372876392
Joints:
- removed joint j1_logo_left
- removed joint j4_left_logo
- added joint j1_logo: type fixed, parent link1, child link1_logo, origin xyz=0 0 0 rpy=0 0 0, axis 0 0 0
- added joint j4_logo_left: type fixed, parent link4, child link4_logo_left, origin xyz=0.44454 0 0 rpy=-2.7775E-05 0 0, axis 0 0 0
- joint j2: limit lower=0 upper=0 effort=0 velocity=0 -> lower=-1.2217 upper=3.1416 effort=100 velocity=1; origin xyz=0.15 0.0815 0.23902 rpy=1.5708 0 1.5708 -> xyz=0.15 0.0815 0.239 rpy=1.5708 0 1.5708
- joint j3: origin xyz=0 0 0.61 rpy=0 0.0082054 -1.5708 -> xyz=0 0 0.61 rpy=0 0 -1.5708
- joint j4: origin xyz=0.2333 -0.0815 0.14192 rpy=0 -0.0082054 0 -> xyz=0.23446 -0.0815 0.14 rpy=0 0 0
- joint j4_logo_right: child link4_right_logo -> link4_logo_right; origin xyz=0.444539076030978 0 0 rpy=0 0 0 -> xyz=0.44454 0.01 0 rpy=-2.7775E-05 0 0
- joint j5: limit lower=-3.14 upper=3.14 effort=10 velocity=1 -> lower=-2.4435 upper=2.4435 effort=0 velocity=0; origin xyz=0.44454 0 0 rpy=0 0 0 -> xyz=0.44454 0.01 0 rpy=0 0 0
- joint j6: origin xyz=0.082 0 0 rpy=0 0 0 -> xyz=0.082 -0.01 0 rpy=0 0 0

Commit message: Update MZ12H.urdf

File: urdf/MZ12H.urdf (robot description, URDF)
Before this commit: robot MZ12H, 10 links, 9 joints
Joints:
- joint j2: axis 0 -1 0 -> 1 0 0

Commit message: fa

File: urdf/MZ12H.urdf (robot description, URDF)
Before this commit: robot MZ12H, 10 links, 9 joints
Joints:
- joint j2: axis 1 0 0 -> 0 -1 0

Commit message: s

File: urdf/MZ12H.urdf (robot description, URDF)
Before this commit: robot MZ12H, 10 links, 9 joints
Joints:
- joint j2: axis 0 -1 0 -> 0 0 1

Commit message: Update MZ12H.urdf

File: urdf/MZ12H.urdf (robot description, URDF)
Before this commit: robot MZ12H, 10 links, 9 joints
Joints:
- joint j2: axis 0 0 1 -> -1 0 0; limit lower=-1.2217 upper=3.1416 effort=100 velocity=1 -> lower=-1.2217 upper=3.1416 effort=0 velocity=0
